File: C13.kicad_pcb (KiCad board)
At the start: 2 copper layers, 80 x 40.1 mm, 120 parts, among them IC1 74HC595BQ,115, IC2 MPM3610AGQV-P, IC9 THVD1450DRBR, J1 V24, J2 Conn_02x04, J3 Conn_02x03, J4 Screw_Terminal_01x04, J5 UDPI, J6 Screw_Terminal_01x04, J7 Screw_Terminal_01x02, K1 G6K-2, Q1 BC848W, Q5 BC857BS, U1 AVR-64DA48, U10 INA181-A1, U11 INA381, U12 INA381, U13 INA181-A1, U14 INA381, U15 INA381, U16 INA181-A4, U2 MIC5235-3.3, U3 INA181-A1, U4 KA78M05_TO252, U5 INA381, U6 INA381, U7 INA181-A1, U8 INA381-A2, U9 INA381, X1 ASE-xxxMHz

Commit message: Initial commit
Parts:
- IC1: footprint SamacSys:74HC595BQ115 -> RTB:74HC595BQ115
- IC2: footprint SamacSys:MPM3610AGQVP -> RTB:MPM3610AGQVP
- IC9: footprint SamacSys:SON65P300X300X100-9N-D -> RTB:SON65P300X300X100-9N-D
- J2: footprint _Samac:1725711 -> RTB:1725711
