File: C13.kicad_pcb (KiCad board)
At the start: 2 copper layers, 80 x 40.1 mm, 119 parts, among them IC1 74HC595BQ,115, IC2 MPM3610AGQV, IC9 THVD1450DRBR, J1 V24, J2 DCC connector, J3 EDG connector, J4 Power Daisy Chain, J5 UDPI, J6 Power Daisy Chain, J7 Power Output, K1 G6K-2, Q1 BC848, Q3 BC857BS, U1 AVR-64DA48, U10 INA181-A1, U11 INA381, U12 INA381, U13 INA181-A1, U14 INA381, U15 INA381, U16 INA181-A4, U2 MIC5235-3.3, U3 INA181-A1, U5 INA381, U6 INA381, U7 INA181-A1, U8 INA381, U9 INA381, X1 ASE-xxxMHz

Commit message: mod: part #
Parts:
- added C9: 1u, Capacitor_SMD:C_0805_2012Metric, B.Cu at (69.8, -23.6)
- added D26: Schottky, Diode_SMD:D_0603_1608Metric, B.Cu at (70.6, -20.4)
- added D27: Schottky, Diode_SMD:D_0603_1608Metric, B.Cu at (69.1, -20.4)
Connections:
- net Net-(U1-PD4) renamed PD4
- net Net-(U1-PD5) renamed PD5
Routing:
- net +3V3: track 181.4 -> 184.4 mm
- net PD5: track 28.5 -> 30.2 mm
- net PD4: track 29.2 -> 30.5 mm
- net GND: vias 30 -> 31
Other:
- board text added: "C13.3"
- board text removed: "C13.2"
