File: C13cpu.kicad_sch (KiCad schematic)
At the start: 42 parts, among them IC1 74HC595BQ,115, IC9 THVD1450DRBR, J1 V24, J5 UDPI, U1 AVR-64DA48, X1 ASE-xxxMHz

Commit message: mod: conversion to KiCad 9
Parts:
- R24, R26: LCSC Part # C21190 -> C11702
Changed lines of the file:
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@@
 			)
 		)
-		(property "Description" "-55℃~+155℃ 100mW 1kΩ 75V Thick Film Resistor ±1% ±100ppm/℃ 0603 Chip Resistor - Surface Mount ROHS"
+		(property "Description" "-55℃~+155℃ 1kΩ 50V 62.5mW Thick Film Resistor ±1% ±100ppm/℃ 0402 Chip Resistor - Surface Mount ROHS"
 			(at 91.44 82.55 0)
 			(effects
@@
 			)
 		)
-		(property "LCSC Part #" "C21190"
+		(property "LCSC Part #" "C11702"
 			(at 91.44 82.55 0)
 			(effects
@@
 			)
 		)
-		(property "Description" "-55℃~+155℃ 100mW 1kΩ 75V Thick Film Resistor ±1% ±100ppm/℃ 0603 Chip Resistor - Surface Mount ROHS"
+		(property "Description" "-55℃~+155℃ 1kΩ 50V 62.5mW Thick Film Resistor ±1% ±100ppm/℃ 0402 Chip Resistor - Surface Mount ROHS"
 			(at 40.64 109.22 0)
 			(effects
@@
 			)
 		)
-		(property "LCSC Part #" "C21190"
+		(property "LCSC Part #" "C11702"
 			(at 40.64 109.22 0)
 			(effects

Commit message: mod: part #
Parts:
- added C9: 1u, Capacitor_SMD:C_0805_2012Metric, symbol Device:C_Small
- added D26, D27: Schottky, Diode_SMD:D_0603_1608Metric, symbol Device:D
Connections:
- net +3V3: now also C9.1, D26.1 (K), D27.1 (K)
- net GND: now also C9.2
- net PD4: now reaches R7.2, U1.24 (PD4)
- net PD4: now also D27.2 (A)
- net PD5: now reaches R8.2, U1.25 (PD5)
- net PD5: now also D26.2 (A)
Other:
- note added: "Rev 3: added D26/D27"
- moved on the sheet: C11, J1, J5, R7, R8, X1
