File: C13rcm.kicad_sch (KiCad schematic)
At the start: 41 parts, among them Q3 BC857BS, U10 INA181-A1, U11 INA381, U12 INA381, U13 INA181-A1, U14 INA381, U15 INA381, U3 INA181-A1, U5 INA381, U6 INA381, U7 INA181-A1, U8 INA381, U9 INA381

Commit message: mod: part #
Parts:
- U11, U12, U14, U15, U5, U6, U8, U9: value INA381 -> INA381A2; LCSC Part # C544574 -> C2155688
Changed lines of the file:
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@@
 		(title "RTB C13 Module")
 		(date "2025-10-14")
-		(rev "2")
+		(rev "3")
 		(company "Frank Schumacher")
 		(comment 1 "Track Sensor")
@@
 			)
 		)
-		(property "Value" "INA381"
+		(property "Value" "INA381A2"
 			(at 99.06 50.8 0)
 			(effects
@@
 			)
 		)
-		(property "LCSC Part #" "C544574"
+		(property "LCSC Part #" "C2155688"
 			(at 93.98 46.99 0)
 			(effects
@@
 			)
 		)
-		(property "Value" "INA381"
+		(property "Value" "INA381A2"
 			(at 133.35 50.8 0)
 			(effects
@@
 			)
 		)
-		(property "LCSC Part #" "C544574"
+		(property "LCSC Part #" "C2155688"
 			(at 128.27 46.99 0)
 			(effects
@@
 			)
 		)
-		(property "Value" "INA381"
+		(property "Value" "INA381A2"
 			(at 99.06 104.14 0)
 			(effects
@@
 			)
 		)
-		(property "LCSC Part #" "C544574"
+		(property "LCSC Part #" "C2155688"
 			(at 93.98 100.33 0)
 			(effects
@@
 			)
 		)
-		(property "Value" "INA381"
+		(property "Value" "INA381A2"
 			(at 133.35 104.14 0)
 			(effects
@@
 			)
 		)
-		(property "LCSC Part #" "C544574"
+		(property "LCSC Part #" "C2155688"
 			(at 128.27 100.33 0)
 			(effects
@@
 			)
 		)
-		(property "Value" "INA381"
+		(property "Value" "INA381A2"
 			(at 229.87 50.8 0)
 			(effects
@@
 			)
 		)
-		(property "LCSC Part #" "C544574"
+		(property "LCSC Part #" "C2155688"
 			(at 224.79 46.99 0)
 			(effects
@@
 			)
 		)
-		(property "Value" "INA381"
+		(property "Value" "INA381A2"
 			(at 264.16 50.8 0)
 			(effects
@@
 			)
 		)
-		(property "LCSC Part #" "C544574"
+		(property "LCSC Part #" "C2155688"
 			(at 259.08 46.99 0)
 			(effects
@@
 			)
 		)
-		(property "Value" "INA381"
+		(property "Value" "INA381A2"
 			(at 229.87 104.14 0)
 			(effects
@@
 			)
 		)
-		(property "LCSC Part #" "C544574"
+		(property "LCSC Part #" "C2155688"
 			(at 224.79 100.33 0)
 			(effects
@@
 			)
 		)
-		(property "Value" "INA381"
+		(property "Value" "INA381A2"
 			(at 264.16 104.14 0)
 			(effects
@@
 			)
 		)
-		(property "LCSC Part #" "C544574"
+		(property "LCSC Part #" "C2155688"
 			(at 259.08 100.33 0)
 			(effects
